Commit message: removed package dependencies

File: urdf/warebot_v3.urdf (robot description, URDF)
Before this commit: robot warebot_v3, 10 links, 9 joints
Links:
- link FL_l_tube: geometry collision mesh filename=package://gantry_assembly_v2/meshes_warebot/FL_l_tube.STL; visual mesh filename=package://gantry_assembly_v2/meshes_warebot/FL_l_tube.STL
- link FL_wheel: geometry collision mesh filename=package://gantry_assembly_v2/meshes_warebot/FL_wheel.STL; visual mesh filename=package://gantry_assembly_v2/meshes_warebot/FL_wheel.STL
- link FR_l_tube: geometry collision mesh filename=package://gantry_assembly_v2/meshes_warebot/FR_l_tube.STL; visual mesh filename=package://gantry_assembly_v2/meshes_warebot/FR_l_tube.STL
- link FR_wheel: geometry collision mesh filename=package://gantry_assembly_v2/meshes_warebot/FR_wheel.STL; visual mesh filename=package://gantry_assembly_v2/meshes_warebot/FR_wheel.STL
- link RL_l_tube: geometry collision mesh filename=package://gantry_assembly_v2/meshes_warebot/RL_l_tube.STL; visual mesh filename=package://gantry_assembly_v2/meshes_warebot/RL_l_tube.STL
- link RL_wheel: geometry collision mesh filename=package://gantry_assembly_v2/meshes_warebot/RL_wheel.STL; visual mesh filename=package://gantry_assembly_v2/meshes_warebot/RL_wheel.STL
- link RR_l_tube: geometry collision mesh filename=package://gantry_assembly_v2/meshes_warebot/RR_l_tube.STL; visual mesh filename=package://gantry_assembly_v2/meshes_warebot/RR_l_tube.STL
- link RR_wheel: geometry collision mesh filename=package://gantry_assembly_v2/meshes_warebot/RR_wheel.STL; visual mesh filename=package://gantry_assembly_v2/meshes_warebot/RR_wheel.STL
- link chassis: geometry collision mesh filename=package://gantry_assembly_v2/meshes_warebot/chassis.STL; visual mesh filename=package://gantry_assembly_v2/meshes_warebot/chassis.STL
