Commit message: robot arm package dependency removed

File: urdf/tu_nguyen.urdf (robot description, URDF)
Before this commit: robot tu_nguyen, 9 links, 8 joints
Links:
- link base_link: geometry collision mesh filename=package://gantry_assembly_v2/meshes_arm/base_link.STL; visual mesh filename=package://gantry_assembly_v2/meshes_arm/base_link.STL
- link link_1: geometry collision mesh filename=package://gantry_assembly_v2/meshes_arm/link_1.STL; visual mesh filename=package://gantry_assembly_v2/meshes_arm/link_1.STL
- link link_2: geometry collision mesh filename=package://gantry_assembly_v2/meshes_arm/link_2.STL; visual mesh filename=package://gantry_assembly_v2/meshes_arm/link_2.STL
- link link_3: geometry collision mesh filename=package://gantry_assembly_v2/meshes_arm/link_3.STL; visual mesh filename=package://gantry_assembly_v2/meshes_arm/link_3.STL
- link link_4: geometry collision mesh filename=package://gantry_assembly_v2/meshes_arm/link_4.STL; visual mesh filename=package://gantry_assembly_v2/meshes_arm/link_4.STL
- link link_51: geometry collision mesh filename=package://gantry_assembly_v2/meshes_arm/link_51.STL; visual mesh filename=package://gantry_assembly_v2/meshes_arm/link_51.STL
- link link_52: geometry collision mesh filename=package://gantry_assembly_v2/meshes_arm/link_52.STL; visual mesh filename=package://gantry_assembly_v2/meshes_arm/link_52.STL
